Commit message: fix: change ur setting

File: crisp_controllers_robot_demos/config/ur/ur_single.urdf.xacro (robot description, xacro)
@@ -1,27 +1,18 @@
 <?xml version='1.0' encoding='utf-8'?>
 <robot xmlns:xacro="http://www.ros.org/wiki/xacro" name="ur">
-  <!-- UR kinematic/visual description (from ur_description package) -->
   <xacro:include filename="$(find ur_description)/urdf/ur_macro.xacro"/>
-  <!-- Custom crisp controllers ROS2 control macro -->
-  <xacro:include filename="$(find crisp_controllers_robot_demos)/config/ur/ur.ros2_control.urdf.xacro"/>
-  <!-- Robot type: ur3, ur3e, ur5, ur5e, ur10, ur10e, ur16e, ur20, etc. -->
-  <xacro:arg name="ur_type" default="ur5e"/>
-  <!-- IP address of the physical robot (ignored when use_fake_hardware=true) -->
-  <xacro:arg name="robot_ip" default="192.168.56.101"/>
-  <!-- Use mock hardware for simulation instead of real robot -->
-  <xacro:arg name="use_fake_hardware" default="false"/>
-  <!-- Optional joint/link name prefix (without trailing underscore) -->
-  <xacro:arg name="tf_prefix" default=""/>
+  <xacro:arg name="ur_type"             default="ur5e"/>
+  <xacro:arg name="robot_ip"            default="192.168.56.101"/>
+  <xacro:arg name="use_fake_hardware"   default="false"/>
+  <xacro:arg name="tf_prefix"           default=""/>
+  <xacro:arg name="script_filename"
+    default="$(find ur_robot_driver)/resources/ros_control.urscript"/>
+  <xacro:arg name="output_recipe_filename"
+    default="$(find ur_robot_driver)/resources/rtde_output_recipe.txt"/>
+  <xacro:arg name="input_recipe_filename"
+    default="$(find ur_robot_driver)/resources/rtde_input_recipe.txt"/>
   <xacro:property name="ur_type_val"   value="${xacro.arg('ur_type')}"/>
   <xacro:property name="tf_prefix_val" value="${xacro.arg('tf_prefix')}"/>
-  <xacro:property name="kinematics_file"
-    value="$(find ur_description)/config/${ur_type_val}/default_kinematics.yaml"/>
-  <!-- Fixed world root link -->
   <link name="world"/>
-  <!--
-    UR robot description: visuals + kinematics only.
-    generate_ros2_control_tag="false" prevents ur_description from inserting its own
-    ros2_control block so that our custom crisp-controller block (below) is the only one.
-  -->
   <xacro:ur_robot
     name="${ur_type_val}"
@@ -29,16 +20,14 @@
     parent="world"
     joint_limits_parameters_file="$(find ur_description)/config/${ur_type_val}/joint_limits.yaml"
-    kinematics_parameters_file="${kinematics_file}"
+    kinematics_parameters_file="$(find ur_description)/config/${ur_type_val}/default_kinematics.yaml"
     physical_parameters_file="$(find ur_description)/config/${ur_type_val}/physical_parameters.yaml"
     visual_parameters_file="$(find ur_description)/config/${ur_type_val}/visual_parameters.yaml"
-    generate_ros2_control_tag="false">
+    robot_ip="$(arg robot_ip)"
+    use_fake_hardware="$(arg use_fake_hardware)"
+    script_filename="$(arg script_filename)"
+    output_recipe_filename="$(arg output_recipe_filename)"
+    input_recipe_filename="$(arg input_recipe_filename)"
+    generate_ros2_control_tag="true">
     <origin xyz="0 0 0" rpy="0 0 0"/>
   </xacro:ur_robot>
-  <!-- Crisp controllers hardware interface -->
-  <xacro:ur_arm_ros2_control
-    name="${ur_type_val}"
-    robot_ip="$(arg robot_ip)"
-    use_fake_hardware="$(arg use_fake_hardware)"
-    tf_prefix="${tf_prefix_val}"
-    kinematics_parameters_file="${kinematics_file}"/>
 </robot>
