Commit message: Make UR xacros distro-aware for generate_ros2_control_tag
ur_description's ur_robot macro was refactored between Humble and Jazzy:
- Humble's macro also emits a <ros2_control> block and accepts
  generate_ros2_control_tag (we set it false to suppress the placeholder
  block and use the custom ur_arm_ros2_control / MuJoCo systems instead).
- Jazzy's macro is kinematic-only: it never emits ros2_control and has no
  generate_ros2_control_tag parameter, so passing it aborts the launch with
  "Invalid parameter generate_ros2_control_tag".

Branch the ur_robot call on $(env ROS_DISTRO) in all three UR description
xacros (ur_single, ur_single_robotiq, ur_single_mujoco): keep the attribute
on Humble, omit it on Jazzy+. All other attributes are accepted by both
macro versions, so only that one attribute differs between branches.

Co-Authored-By: Claude Opus 4.8 <noreply@anthropic.com>
Claude-Session: https://claude.ai/code/session_01LwcanisLQ82BqUjDtqM6DT

File: crisp_controllers_robot_demos/config/ur/ur_single.urdf.xacro (robot description, xacro)
@@ -18,18 +18,38 @@
   <xacro:property name="tf_prefix_val" value="${xacro.arg('tf_prefix')}"/>
   <link name="world"/>
-  <!-- generate_ros2_control_tag="false": the apt ur_description macro does not honour
-       script_filename/recipe params and produces a to_be_filled_by_ur_robot_driver
-       placeholder. The custom ur_arm_ros2_control macro below embeds the correct paths. -->
-  <xacro:ur_robot
-    name="${ur_type_val}"
-    tf_prefix="${tf_prefix_val}"
-    parent="world"
-    joint_limits_parameters_file="$(find ur_description)/config/${ur_type_val}/joint_limits.yaml"
-    kinematics_parameters_file="$(arg kinematics_parameters_file)"
-    physical_parameters_file="$(find ur_description)/config/${ur_type_val}/physical_parameters.yaml"
-    visual_parameters_file="$(find ur_description)/config/${ur_type_val}/visual_parameters.yaml"
-    generate_ros2_control_tag="false">
-    <origin xyz="0 0 0" rpy="0 0 0"/>
-  </xacro:ur_robot>
+  <!-- ur_description's ur_robot macro differs by distro:
+       - Humble: also emits a <ros2_control> block. We suppress it with
+         generate_ros2_control_tag="false" because that block does not honour
+         script_filename/recipe params (it emits a to_be_filled_by_ur_robot_driver
+         placeholder); the custom ur_arm_ros2_control macro below embeds the real paths.
+       - Jazzy+: the macro is kinematic-only and has no generate_ros2_control_tag
+         parameter, so passing it raises 'Invalid parameter generate_ros2_control_tag'.
+       Branch on ROS_DISTRO so the same file works on both. -->
+  <xacro:arg name="ros_distro" default="$(env ROS_DISTRO)"/>
+  <xacro:if value="${xacro.arg('ros_distro') == 'humble'}">
+    <xacro:ur_robot
+      name="${ur_type_val}"
+      tf_prefix="${tf_prefix_val}"
+      parent="world"
+      joint_limits_parameters_file="$(find ur_description)/config/${ur_type_val}/joint_limits.yaml"
+      kinematics_parameters_file="$(arg kinematics_parameters_file)"
+      physical_parameters_file="$(find ur_description)/config/${ur_type_val}/physical_parameters.yaml"
+      visual_parameters_file="$(find ur_description)/config/${ur_type_val}/visual_parameters.yaml"
+      generate_ros2_control_tag="false">
+      <origin xyz="0 0 0" rpy="0 0 0"/>
+    </xacro:ur_robot>
+  </xacro:if>
+  <xacro:unless value="${xacro.arg('ros_distro') == 'humble'}">
+    <xacro:ur_robot
+      name="${ur_type_val}"
+      tf_prefix="${tf_prefix_val}"
+      parent="world"
+      joint_limits_parameters_file="$(find ur_description)/config/${ur_type_val}/joint_limits.yaml"
+      kinematics_parameters_file="$(arg kinematics_parameters_file)"
+      physical_parameters_file="$(find ur_description)/config/${ur_type_val}/physical_parameters.yaml"
+      visual_parameters_file="$(find ur_description)/config/${ur_type_val}/visual_parameters.yaml">
+      <origin xyz="0 0 0" rpy="0 0 0"/>
+    </xacro:ur_robot>
+  </xacro:unless>
   <xacro:ur_arm_ros2_control
     name="${ur_type_val}"

File: crisp_controllers_robot_demos/config/ur/ur_single_mujoco.urdf.xacro (robot description, xacro)
@@ -14,17 +14,38 @@
   <xacro:property name="tf_prefix_val" value="${xacro.arg('tf_prefix')}"/>
   <link name="world"/>
-  <!-- Kinematic/visual URDF only — generate_ros2_control_tag=false because the
-       hardware is the MuJoCo simulator below, not the UR driver/mock. -->
-  <xacro:ur_robot
-    name="${ur_type_val}"
-    tf_prefix="${tf_prefix_val}"
-    parent="world"
-    joint_limits_parameters_file="$(find ur_description)/config/${ur_type_val}/joint_limits.yaml"
-    kinematics_parameters_file="$(arg kinematics_parameters_file)"
-    physical_parameters_file="$(find ur_description)/config/${ur_type_val}/physical_parameters.yaml"
-    visual_parameters_file="$(find ur_description)/config/${ur_type_val}/visual_parameters.yaml"
-    generate_ros2_control_tag="false">
-    <origin xyz="0 0 0" rpy="0 0 0"/>
-  </xacro:ur_robot>
+  <!-- Kinematic/visual URDF only; the hardware is the MuJoCo simulator below, not
+       the UR driver/mock. ur_description's ur_robot macro differs by distro:
+       - Humble: also emits a <ros2_control> block, suppressed with
+         generate_ros2_control_tag="false" so it does not clash with the MuJoCo
+         ros2_control system defined below.
+       - Jazzy+: the macro is kinematic-only and has no generate_ros2_control_tag
+         parameter, so passing it raises 'Invalid parameter generate_ros2_control_tag'.
+       Branch on ROS_DISTRO so the same file works on both. -->
+  <xacro:arg name="ros_distro" default="$(env ROS_DISTRO)"/>
+  <xacro:if value="${xacro.arg('ros_distro') == 'humble'}">
+    <xacro:ur_robot
+      name="${ur_type_val}"
+      tf_prefix="${tf_prefix_val}"
+      parent="world"
+      joint_limits_parameters_file="$(find ur_description)/config/${ur_type_val}/joint_limits.yaml"
+      kinematics_parameters_file="$(arg kinematics_parameters_file)"
+      physical_parameters_file="$(find ur_description)/config/${ur_type_val}/physical_parameters.yaml"
+      visual_parameters_file="$(find ur_description)/config/${ur_type_val}/visual_parameters.yaml"
+      generate_ros2_control_tag="false">
+      <origin xyz="0 0 0" rpy="0 0 0"/>
+    </xacro:ur_robot>
+  </xacro:if>
+  <xacro:unless value="${xacro.arg('ros_distro') == 'humble'}">
+    <xacro:ur_robot
+      name="${ur_type_val}"
+      tf_prefix="${tf_prefix_val}"
+      parent="world"
+      joint_limits_parameters_file="$(find ur_description)/config/${ur_type_val}/joint_limits.yaml"
+      kinematics_parameters_file="$(arg kinematics_parameters_file)"
+      physical_parameters_file="$(find ur_description)/config/${ur_type_val}/physical_parameters.yaml"
+      visual_parameters_file="$(find ur_description)/config/${ur_type_val}/visual_parameters.yaml">
+      <origin xyz="0 0 0" rpy="0 0 0"/>
+    </xacro:ur_robot>
+  </xacro:unless>
   <!-- MuJoCo-backed arm: effort command + position/velocity/effort state,
        exactly the interface set crisp_mujoco_sim/Simulator requires.

File: crisp_controllers_robot_demos/config/ur/ur_single_robotiq.urdf.xacro (robot description, xacro)
@@ -21,18 +21,38 @@
   <xacro:property name="tf_prefix_val" value="${xacro.arg('tf_prefix')}"/>
   <link name="world"/>
-  <!-- generate_ros2_control_tag="false": the apt ur_description macro does not honour
-       script_filename/recipe params and produces a to_be_filled_by_ur_robot_driver
-       placeholder. The custom ur_arm_ros2_control macro below embeds the correct paths. -->
-  <xacro:ur_robot
-    name="${ur_type_val}"
-    tf_prefix="${tf_prefix_val}"
-    parent="world"
-    joint_limits_parameters_file="$(find ur_description)/config/${ur_type_val}/joint_limits.yaml"
-    kinematics_parameters_file="$(arg kinematics_parameters_file)"
-    physical_parameters_file="$(find ur_description)/config/${ur_type_val}/physical_parameters.yaml"
-    visual_parameters_file="$(find ur_description)/config/${ur_type_val}/visual_parameters.yaml"
-    generate_ros2_control_tag="false">
-    <origin xyz="0 0 0" rpy="0 0 0"/>
-  </xacro:ur_robot>
+  <!-- ur_description's ur_robot macro differs by distro:
+       - Humble: also emits a <ros2_control> block. We suppress it with
+         generate_ros2_control_tag="false" because that block does not honour
+         script_filename/recipe params (it emits a to_be_filled_by_ur_robot_driver
+         placeholder); the custom ur_arm_ros2_control macro below embeds the real paths.
+       - Jazzy+: the macro is kinematic-only and has no generate_ros2_control_tag
+         parameter, so passing it raises 'Invalid parameter generate_ros2_control_tag'.
+       Branch on ROS_DISTRO so the same file works on both. -->
+  <xacro:arg name="ros_distro" default="$(env ROS_DISTRO)"/>
+  <xacro:if value="${xacro.arg('ros_distro') == 'humble'}">
+    <xacro:ur_robot
+      name="${ur_type_val}"
+      tf_prefix="${tf_prefix_val}"
+      parent="world"
+      joint_limits_parameters_file="$(find ur_description)/config/${ur_type_val}/joint_limits.yaml"
+      kinematics_parameters_file="$(arg kinematics_parameters_file)"
+      physical_parameters_file="$(find ur_description)/config/${ur_type_val}/physical_parameters.yaml"
+      visual_parameters_file="$(find ur_description)/config/${ur_type_val}/visual_parameters.yaml"
+      generate_ros2_control_tag="false">
+      <origin xyz="0 0 0" rpy="0 0 0"/>
+    </xacro:ur_robot>
+  </xacro:if>
+  <xacro:unless value="${xacro.arg('ros_distro') == 'humble'}">
+    <xacro:ur_robot
+      name="${ur_type_val}"
+      tf_prefix="${tf_prefix_val}"
+      parent="world"
+      joint_limits_parameters_file="$(find ur_description)/config/${ur_type_val}/joint_limits.yaml"
+      kinematics_parameters_file="$(arg kinematics_parameters_file)"
+      physical_parameters_file="$(find ur_description)/config/${ur_type_val}/physical_parameters.yaml"
+      visual_parameters_file="$(find ur_description)/config/${ur_type_val}/visual_parameters.yaml">
+      <origin xyz="0 0 0" rpy="0 0 0"/>
+    </xacro:ur_robot>
+  </xacro:unless>
   <xacro:ur_arm_ros2_control
     name="${ur_type_val}"
