Commit message: fix: bypass ur_description ros2_control tag; use custom macro to embed script paths
The apt-installed ur_description's xacro:ur_robot macro accepts script_filename,
output_recipe_filename, and input_recipe_filename as arguments but does not honour
them when generate_ros2_control_tag="true" — the internal ur.ros2_control.xacro
template still emits the to_be_filled_by_ur_robot_driver placeholder.

Fix: set generate_ros2_control_tag="false" on xacro:ur_robot and use the project's
own ur_arm_ros2_control macro (ur.ros2_control.urdf.xacro), which explicitly embeds
the correct script_filename and recipe paths as <param> elements. Also adds
headless_mode as a macro parameter (default true) so it flows through from launch args.

https://claude.ai/code/session_01JjRhmpJGHK4phM65xkjwtM

File: crisp_controllers_robot_demos/config/ur/ur.ros2_control.urdf.xacro (robot description, xacro)
@@ -10,8 +10,6 @@
     - tf_prefix: Optional prefix for all joint/link names (without trailing underscore)
     - kinematics_parameters_file: Path to the robot calibration YAML
-  Effort (torque) command interface:
-    Supported on PolyScope X >= 10.12.1 via URScript direct_torque().
-    headless_mode=false: teach pendant runs the External Control program which loads
-    ros_control.urscript. The script receives torque commands via the reverse port.
+    - headless_mode: true → driver pushes URScript over port 30001 (pendant in Remote Control)
+                     false → pendant runs External Control program that loads the script
 -->
 <xacro:macro name="ur_arm_ros2_control"
@@ -20,5 +18,6 @@
              use_fake_hardware
              tf_prefix:=''
-             kinematics_parameters_file">
+             kinematics_parameters_file
+             headless_mode:='true'">
     <xacro:property name="prefix" value="${tf_prefix + '_' if tf_prefix != '' else ''}"/>
     <ros2_control name="${prefix}${name}HardwareInterface" type="system">
@@ -31,5 +30,5 @@
           <param name="output_recipe_filename">$(find ur_robot_driver)/resources/rtde_output_recipe.txt</param>
           <param name="input_recipe_filename">$(find ur_robot_driver)/resources/rtde_input_recipe.txt</param>
-          <param name="headless_mode">false</param>
+          <param name="headless_mode">${headless_mode}</param>
           <!-- Use the upstream urcl bundled script: it has full torque support
                (direct_torque with friction_comp / viscous_scale / coulomb_scale)

File: crisp_controllers_robot_demos/config/ur/ur_single.urdf.xacro (robot description, xacro)
@@ -2,4 +2,5 @@
 <robot xmlns:xacro="http://www.ros.org/wiki/xacro" name="ur">
   <xacro:include filename="$(find ur_description)/urdf/ur_macro.xacro"/>
+  <xacro:include filename="$(find crisp_controllers_robot_demos)/config/ur/ur.ros2_control.urdf.xacro"/>
   <xacro:arg name="ur_type"             default="ur5e"/>
   <xacro:arg name="robot_ip"            default="192.168.56.101"/>
@@ -12,10 +13,4 @@
        Prerequisite: pendant must be in Remote Control mode. -->
   <xacro:arg name="headless_mode"       default="true"/>
-  <xacro:arg name="script_filename"
-    default="$(find ur_client_library)/resources/external_control.urscript"/>
-  <xacro:arg name="output_recipe_filename"
-    default="$(find ur_robot_driver)/resources/rtde_output_recipe.txt"/>
-  <xacro:arg name="input_recipe_filename"
-    default="$(find ur_robot_driver)/resources/rtde_input_recipe.txt"/>
   <xacro:arg name="kinematics_parameters_file"
     default="$(find ur_description)/config/$(arg ur_type)/default_kinematics.yaml"/>
@@ -23,4 +18,7 @@
   <xacro:property name="tf_prefix_val" value="${xacro.arg('tf_prefix')}"/>
   <link name="world"/>
+  <!-- generate_ros2_control_tag="false": the apt ur_description macro does not honour
+       script_filename/recipe params and produces a to_be_filled_by_ur_robot_driver
+       placeholder. The custom ur_arm_ros2_control macro below embeds the correct paths. -->
   <xacro:ur_robot
     name="${ur_type_val}"
@@ -31,12 +29,13 @@
     physical_parameters_file="$(find ur_description)/config/${ur_type_val}/physical_parameters.yaml"
     visual_parameters_file="$(find ur_description)/config/${ur_type_val}/visual_parameters.yaml"
+    generate_ros2_control_tag="false">
+    <origin xyz="0 0 0" rpy="0 0 0"/>
+  </xacro:ur_robot>
+  <xacro:ur_arm_ros2_control
+    name="${ur_type_val}"
     robot_ip="$(arg robot_ip)"
     use_fake_hardware="$(arg use_fake_hardware)"
+    tf_prefix="${tf_prefix_val}"
     headless_mode="$(arg headless_mode)"
-    script_filename="$(arg script_filename)"
-    output_recipe_filename="$(arg output_recipe_filename)"
-    input_recipe_filename="$(arg input_recipe_filename)"
-    generate_ros2_control_tag="true">
-    <origin xyz="0 0 0" rpy="0 0 0"/>
-  </xacro:ur_robot>
+    kinematics_parameters_file="$(arg kinematics_parameters_file)"/>
 </robot>

File: crisp_controllers_robot_demos/config/ur/ur_single_robotiq.urdf.xacro (robot description, xacro)
@@ -3,4 +3,5 @@
   <xacro:include filename="$(find ur_description)/urdf/ur_macro.xacro"/>
   <xacro:include filename="$(find robotiq_description)/urdf/robotiq_2f_140_macro.urdf.xacro"/>
+  <xacro:include filename="$(find crisp_controllers_robot_demos)/config/ur/ur.ros2_control.urdf.xacro"/>
   <xacro:arg name="ur_type"             default="ur5e"/>
   <xacro:arg name="robot_ip"            default="192.168.56.101"/>
@@ -15,10 +16,4 @@
   <!-- Robotiq 2F-140 serial port. USB-to-RS485 adapter on the host. -->
   <xacro:arg name="com_port"            default="/dev/ttyUSB0"/>
-  <xacro:arg name="script_filename"
-    default="$(find ur_client_library)/resources/external_control.urscript"/>
-  <xacro:arg name="output_recipe_filename"
-    default="$(find ur_robot_driver)/resources/rtde_output_recipe.txt"/>
-  <xacro:arg name="input_recipe_filename"
-    default="$(find ur_robot_driver)/resources/rtde_input_recipe.txt"/>
   <xacro:arg name="kinematics_parameters_file"
     default="$(find ur_description)/config/$(arg ur_type)/default_kinematics.yaml"/>
@@ -26,4 +21,7 @@
   <xacro:property name="tf_prefix_val" value="${xacro.arg('tf_prefix')}"/>
   <link name="world"/>
+  <!-- generate_ros2_control_tag="false": the apt ur_description macro does not honour
+       script_filename/recipe params and produces a to_be_filled_by_ur_robot_driver
+       placeholder. The custom ur_arm_ros2_control macro below embeds the correct paths. -->
   <xacro:ur_robot
     name="${ur_type_val}"
@@ -34,13 +32,14 @@
     physical_parameters_file="$(find ur_description)/config/${ur_type_val}/physical_parameters.yaml"
     visual_parameters_file="$(find ur_description)/config/${ur_type_val}/visual_parameters.yaml"
+    generate_ros2_control_tag="false">
+    <origin xyz="0 0 0" rpy="0 0 0"/>
+  </xacro:ur_robot>
+  <xacro:ur_arm_ros2_control
+    name="${ur_type_val}"
     robot_ip="$(arg robot_ip)"
     use_fake_hardware="$(arg use_fake_hardware)"
+    tf_prefix="${tf_prefix_val}"
     headless_mode="$(arg headless_mode)"
-    script_filename="$(arg script_filename)"
-    output_recipe_filename="$(arg output_recipe_filename)"
-    input_recipe_filename="$(arg input_recipe_filename)"
-    generate_ros2_control_tag="true">
-    <origin xyz="0 0 0" rpy="0 0 0"/>
-  </xacro:ur_robot>
+    kinematics_parameters_file="$(arg kinematics_parameters_file)"/>
   <!-- Attach the Robotiq 2F-140 to the UR tool flange (tool0).
        include_ros2_control adds a second hardware system (finger_joint position
