Commit message: Fix UR external-effort: real gripper payload + scale-free calibration
Two coupled corrections so external-effort estimation reflects contact, not
the gripper's own weight:

1. Payload mass. The robotiq_description URDF models only ~0.364 kg of the
   2F-140, but identify_payload (wrist F/T) measured the true gripper+coupling
   at 1.3096 kg, COM in tool0 = (-0.0021, -0.0031, 0.0579) m. Add the
   difference as a lumped inertial at that COM on tool0 in
   ur_single_robotiq.urdf.xacro, so the Pinocchio gravity g(q) accounts for the
   real payload (mass/COM are xacro args; re-run identify_payload if the tool
   changes). Only mass+COM affect gravity torque; the inertia tensor is a
   placeholder.

2. Calibration. Stop least-squares fitting the gravity `scale`: g(q) is the
   physically correct RNEA gravity and must not be rescaled (a fitted gain
   distorts a correct model and was masking the missing payload). Fit only the
   constant per-joint offset = mean(tau - g); scale stays 1.0. Updated
   external_effort.py::fit_calibration, the calibrate node, docstrings and the
   README accordingly.

Co-Authored-By: Claude Opus 4.8 <noreply@anthropic.com>
Claude-Session: https://claude.ai/code/session_01LwcanisLQ82BqUjDtqM6DT

File: crisp_controllers_robot_demos/config/ur/ur_single_robotiq.urdf.xacro (robot description, xacro)
@@ -71,3 +71,32 @@
     <origin xyz="0 0 0" rpy="0 0 0"/>
   </xacro:robotiq_gripper>
+  <!-- Measured payload correction. The robotiq_description URDF models only
+       ~0.364 kg of the 2F-140, but the true gripper + coupling + fingers was
+       measured at 1.3096 kg with COM in tool0 = (-0.0021, -0.0031, 0.0579) m
+       using `ros2 run crisp_controllers_robot_demos identify_payload` (wrist F/T
+       least-squares fit). Add the DIFFERENCE as a lumped mass at the measured
+       COM so the Pinocchio gravity model g(q) - used by external_effort
+       estimation AND any model-based controller reading /robot_description -
+       reflects the real payload. Only mass and COM affect gravity torque; the
+       inertia tensor is a compact placeholder. Re-run identify_payload and update
+       these args if the tool changes. (Placing the supplement at the measured COM
+       assumes the robotiq model's COM ~ the true COM, which holds because the
+       gripper geometry is modeled even though its mass magnitude was too low.) -->
+  <xacro:arg name="gripper_total_mass" default="1.3096"/>
+  <xacro:arg name="gripper_com_x"      default="-0.0021"/>
+  <xacro:arg name="gripper_com_y"      default="-0.0031"/>
+  <xacro:arg name="gripper_com_z"      default="0.0579"/>
+  <link name="${tf_prefix_val}gripper_payload_correction">
+    <inertial>
+      <origin xyz="$(arg gripper_com_x) $(arg gripper_com_y) $(arg gripper_com_z)" rpy="0 0 0"/>
+      <!-- supplement = measured total - the ~0.364 kg the robotiq URDF already models -->
+      <mass value="${$(arg gripper_total_mass) - 0.364}"/>
+      <inertia ixx="1e-4" ixy="0" ixz="0" iyy="1e-4" iyz="0" izz="1e-4"/>
+    </inertial>
+  </link>
+  <joint name="${tf_prefix_val}gripper_payload_correction_joint" type="fixed">
+    <parent link="tool0"/>
+    <child  link="${tf_prefix_val}gripper_payload_correction"/>
+    <origin xyz="0 0 0" rpy="0 0 0"/>
+  </joint>
 </robot>
