Commit message: Rotate the Robotiq an extra -45 deg about Z at the fr3 flange
The mount origin in fr3_single_robotiq.urdf.xacro carried only the -45 deg
about Z of the Franka Hand convention. On this coupling that leaves the
Robotiq 45 deg off, so the flange mount now applies -90 deg (-pi/2) total.

Affects the description loaded by launch_franka_gripper
(franka.launch.py with use_gripper:=true), i.e. the arm-side TF/visual for
the gripper and everything downstream of robotiq_85_base_link
(robotiq_gripper_tcp and fr3_hand_tcp, the CIC end_effector_frame).

The standalone /robotiq_2f85 control description is unchanged: it mounts the
gripper to world and is not part of the arm's TF tree.

Co-Authored-By: Claude Opus 5 <noreply@anthropic.com>
Claude-Session: https://claude.ai/code/session_01AiBNGyJH87B1isfCKmXftt

File: crisp_controllers_robot_demos/config/fr3/fr3_single_robotiq.urdf.xacro (robot description, xacro)
@@ -29,5 +29,8 @@
   <!-- Mounted on the flange (fr3_link8). Adjust the origin to match your
        coupling: the Franka Hand convention rotates the EE by -45 deg about Z,
-       and a coupling kit adds a Z offset. -->
+       and a coupling kit adds a Z offset.
+       This coupling needs a FURTHER -45 deg on top of that convention, so the
+       total yaw is -90 deg (-pi/2) about Z. Measured on the real gripper: with
+       only the -45 deg Franka convention the Robotiq sat 45 deg off. -->
   <!-- include_ros2_control="false": the Robotiq is VISUAL-only in the franka
        URDF (links/TF). Its control lives on a SEPARATE /robotiq
@@ -42,5 +45,5 @@
     com_port="$(arg com_port)"
     include_ros2_control="false">
-    <origin xyz="0 0 0" rpy="0 0 ${-pi/4}"/>
+    <origin xyz="0 0 0" rpy="0 0 ${-pi/2}"/>
   </xacro:robotiq_gripper>
   <!-- Robotiq 2F-85 TCP: 0.1025 m along the approach axis (Z) from the gripper
